File: schematic/flipdot34/flipdot34.kicad_pcb (KiCad board)
At the start: 2 copper layers, 78.7 x 66 mm, 15 parts, among them J1 FlipDot matrix, J2 I2C bus, J3 Config Jumpers, J4 Power 24V, U1 74HC595, U2 74HC595

Commit message: Minor fixes
Routing:
- net Vin: track 217.6 -> 228.1 mm, vias 8 -> 6
- net B1-X: track 24.6 -> 23.2 mm
- net RESET: track 20.4 -> 19.7 mm
- net Net-(A1-Pad13): track 61.5 -> 60.7 mm
Changed lines of the file:
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@@
     (style (thickness 0.15) (arrow_length 1.27) (text_position_mode 0) (extension_height 0.58642) (extension_offset 0.5) keep_text_aligned)
   )
-  (segment (start 134.62 78.74) (end 134.62 96.52) (width 0.5) (layer "B.Cu") (net 5))
-  (segment (start 134.62 96.52) (end 131.954547 96.52) (width 0.5) (layer "B.Cu") (net 5))
+  (segment (start 133.35 96.52) (end 131.954547 96.52) (width 0.5) (layer "B.Cu") (net 5))
+  (segment (start 134.62 95.25) (end 133.35 96.52) (width 0.5) (layer "B.Cu") (net 5))
+  (segment (start 134.62 78.74) (end 134.62 95.25) (width 0.5) (layer "B.Cu") (net 5))
   (segment (start 154.935 119.361549) (end 147.212998 119.361549) (width 0.5) (layer "B.Cu") (net 6))
   (segment (start 147.212998 119.361549) (end 147.194547 119.38) (width 0.5) (layer "B.Cu") (net 6))
@@
   (segment (start 91.44 91.44) (end 91.44 86.36) (width 0.5) (layer "F.Cu") (net 22))
   (segment (start 123.19 83.82) (end 142.24 83.82) (width 0.5) (layer "F.Cu") (net 22))
-  (segment (start 143.51 129.54) (end 143.51 100.33) (width 0.5) (layer "F.Cu") (net 22))
   (via (at 123.19 83.82) (size 1.4) (drill 0.4) (layers "F.Cu" "B.Cu") (net 22))
   (via (at 91.44 91.44) (size 1.4) (drill 0.4) (layers "F.Cu" "B.Cu") (net 22))
-  (via (at 143.51 129.54) (size 1.4) (drill 0.4) (layers "F.Cu" "B.Cu") (net 22))
   (via (at 91.44 111.76) (size 1.4) (drill 0.4) (layers "F.Cu" "B.Cu") (net 22))
-  (via (at 143.51 100.33) (size 1.4) (drill 0.4) (layers "F.Cu" "B.Cu") (net 22))
   (via (at 142.24 83.82) (size 1.4) (drill 0.4) (layers "F.Cu" "B.Cu") (free) (net 22))
   (via (at 91.44 86.36) (size 1.4) (drill 0.4) (layers "F.Cu" "B.Cu") (net 22))
   (via (at 91.44 97.79) (size 1.4) (drill 0.4) (layers "F.Cu" "B.Cu") (net 22))
+  (segment (start 139.7 133.35) (end 143.51 129.54) (width 0.8) (layer "B.Cu") (net 22))
   (segment (start 95.265 86.345) (end 91.455 86.345) (width 0.5) (layer "B.Cu") (net 22))
-  (segment (start 144.78 99.06) (end 143.51 100.33) (width 0.5) (layer "B.Cu") (net 22))
+  (segment (start 160.02 120.65) (end 160.02 104.182894) (width 0.8) (layer "B.Cu") (net 22))
   (segment (start 91.4 111.8) (end 91.44 111.76) (width 0.5) (layer "B.Cu") (net 22))
+  (segment (start 93.98 132.08) (end 95.25 133.35) (width 0.8) (layer "B.Cu") (net 22))
   (segment (start 91.4 97.75) (end 91.44 97.79) (width 0.5) (layer "B.Cu") (net 22))
-  (segment (start 93.98 125.73) (end 93.98 132.08) (width 0.8) (layer "B.Cu") (net 22))
   (segment (start 91.455 86.345) (end 91.44 86.36) (width 0.5) (layer "B.Cu") (net 22))
-  (segment (start 119.38 133.35) (end 139.7 133.35) (width 0.8) (layer "B.Cu") (net 22))
+  (segment (start 156.129521 124.540479) (end 160.02 120.65) (width 0.8) (layer "B.Cu") (net 22))
   (segment (start 142.24 78.74) (end 142.24 83.82) (width 0.5) (layer "B.Cu") (net 22))
   (segment (start 147.237441 99.102894) (end 147.194547 99.06) (width 0.5) (layer "B.Cu") (net 22))
   (segment (start 149.86 78.74) (end 154.94 83.82) (width 0.5) (layer "B.Cu") (net 22))
   (segment (start 91.4 93.98) (end 91.4 97.75) (width 0.8) (layer "B.Cu") (net 22))
+  (segment (start 93.98 125.73) (end 93.98 132.08) (width 0.8) (layer "B.Cu") (net 22))
   (segment (start 91.4 93.98) (end 95.25 93.98) (width 0.8) (layer "B.Cu") (net 22))
-  (segment (start 91.4 119.38) (end 91.4 123.15) (width 0.8) (layer "B.Cu") (net 22))
   (segment (start 91.4 119.38) (end 91.4 111.8) (width 0.8) (layer "B.Cu") (net 22))
   (segment (start 91.4 91.48) (end 91.44 91.44) (width 0.5) (layer "B.Cu") (net 22))
-  (segment (start 147.194547 99.06) (end 144.78 99.06) (width 0.5) (layer "B.Cu") (net 22))
+  (segment (start 91.4 123.15) (end 93.98 125.73) (width 0.8) (layer "B.Cu") (net 22))
   (segment (start 91.4 119.38) (end 95.265 119.38) (width 0.5) (layer "B.Cu") (net 22))
   (segment (start 117.3575 83.82) (end 123.19 83.82) (width 0.5) (layer "B.Cu") (net 22))
   (segment (start 154.94 99.102894) (end 147.237441 99.102894) (width 0.5) (layer "B.Cu") (net 22))
-  (segment (start 92.71 124.46) (end 93.98 125.73) (width 0.8) (layer "B.Cu") (net 22))
   (segment (start 144.78 78.74) (end 149.86 78.74) (width 0.5) (layer "B.Cu") (net 22))
   (segment (start 142.24 78.74) (end 144.78 78.74) (width 0.5) (layer "B.Cu") (net 22))
   (segment (start 154.94 83.82) (end 154.94 86.36) (width 0.5) (layer "B.Cu") (net 22))
+  (segment (start 153.589521 124.540479) (end 156.129521 124.540479) (width 0.8) (layer "B.Cu") (net 22))
   (segment (start 154.94 86.36) (end 154.94 99.102894) (width 0.5) (layer "B.Cu") (net 22))
+  (segment (start 95.25 133.35) (end 139.7 133.35) (width 0.8) (layer "B.Cu") (net 22))
   (segment (start 114.8175 83.82) (end 117.3575 83.82) (width 0.5) (layer "B.Cu") (net 22))
   (segment (start 95.25 93.98) (end 95.265 93.965) (width 0.5) (layer "B.Cu") (net 22))
-  (segment (start 93.98 132.08) (end 95.25 133.35) (width 0.8) (layer "B.Cu") (net 22))
-  (segment (start 95.25 133.35) (end 119.38 133.35) (width 0.8) (layer "B.Cu") (net 22))
-  (segment (start 139.7 133.35) (end 143.51 129.54) (width 0.8) (layer "B.Cu") (net 22))
+  (segment (start 160.02 104.182894) (end 154.94 99.102894) (width 0.8) (layer "B.Cu") (net 22))
+  (segment (start 143.51 129.54) (end 148.59 129.54) (width 0.8) (layer "B.Cu") (net 22))
+  (segment (start 91.4 119.38) (end 91.4 123.15) (width 0.8) (layer "B.Cu") (net 22))
   (segment (start 91.44 111.76) (end 95.265 111.76) (width 0.5) (layer "B.Cu") (net 22))
+  (segment (start 148.59 129.54) (end 153.589521 124.540479) (width 0.8) (layer "B.Cu") (net 22))
   (segment (start 91.4 93.98) (end 91.4 91.48) (width 0.8) (layer "B.Cu") (net 22))
-  (segment (start 91.4 123.15) (end 92.71 124.46) (width 0.8) (layer "B.Cu") (net 22))
   (segment (start 128.27 119.38) (end 120.65 111.76) (width 0.5) (layer "B.Cu") (net 23))
   (segment (start 131.954547 119.38) (end 128.27 119.38) (width 0.5) (layer "B.Cu") (net 23))
   (segment (start 120.65 111.76) (end 117.3575 111.76) (width 0.5) (layer "B.Cu") (net 23))
-  (segment (start 124.46 124.46) (end 99.06 124.46) (width 0.5) (layer "B.Cu") (net 25))
-  (segment (start 97.79 123.19) (end 97.79 114.3) (width 0.5) (layer "B.Cu") (net 25))
+  (segment (start 131.954547 121.92) (end 134.62 121.92) (width 0.5) (layer "B.Cu") (net 25))
+  (segment (start 129.54 129.54) (end 124.46 124.46) (width 0.5) (layer "B.Cu") (net 25))
+  (segment (start 96.52 114.3) (end 95.265 114.3) (width 0.5) (layer "B.Cu") (net 25))
+  (segment (start 133.35 129.54) (end 129.54 129.54) (width 0.5) (layer "B.Cu") (net 25))
   (segment (start 135.89 127) (end 133.35 129.54) (width 0.5) (layer "B.Cu") (net 25))
   (segment (start 134.62 121.92) (end 135.89 123.19) (width 0.5) (layer "B.Cu") (net 25))
-  (segment (start 133.35 129.54) (end 129.54 129.54) (width 0.5) (layer "B.Cu") (net 25))
-  (segment (start 97.79 114.3) (end 95.265 114.3) (width 0.5) (layer "B.Cu") (net 25))
-  (segment (start 129.54 129.54) (end 124.46 124.46) (width 0.5) (layer "B.Cu") (net 25))
+  (segment (start 97.79 123.19) (end 97.79 115.57) (width 0.5) (layer "B.Cu") (net 25))
+  (segment (start 97.79 115.57) (end 96.52 114.3) (width 0.5) (layer "B.Cu") (net 25))
+  (segment (start 124.46 124.46) (end 99.06 124.46) (width 0.5) (layer "B.Cu") (net 25))
+  (segment (start 135.89 123.19) (end 135.89 127) (width 0.5) (layer "B.Cu") (net 25))
   (segment (start 99.06 124.46) (end 97.79 123.19) (width 0.5) (layer "B.Cu") (net 25))
-  (segment (start 131.954547 121.92) (end 134.62 121.92) (width 0.5) (layer "B.Cu") (net 25))
-  (segment (start 135.89 123.19) (end 135.89 127) (width 0.5) (layer "B.Cu") (net 25))
   (segment (start 129.54 124.46) (end 127 121.92) (width 0.5) (layer "B.Cu") (net 26))
   (segment (start 101.6 121.92) (end 100.33 120.65) (width 0.5) (layer "B.Cu") (net 26))
@@
   (segment (start 102.885 93.965) (end 114.8025 93.965) (width 0.5) (layer "B.Cu") (net 33))
   (segment (start 114.8025 93.965) (end 114.8175 93.98) (width 0.5) (layer "B.Cu") (net 33))
-  (segment (start 97.79 96.52) (end 109.22 96.52) (width 0.5) (layer "F.Cu") (net 34))
+  (segment (start 98.9805 96.52) (end 109.22 96.52) (width 0.5) (layer "F.Cu") (net 34))
   (via (at 109.22 96.52) (size 1.4) (drill 0.4) (layers "F.Cu" "B.Cu") (net 34))
-  (via (at 97.79 96.52) (size 1.4) (drill 0.4) (layers "F.Cu" "B.Cu") (net 34))
-  (segment (start 97.775 91.425) (end 97.79 91.44) (width 0.5) (layer "B.Cu") (net 34))
-  (segment (start 95.265 91.425) (end 97.775 91.425) (width 0.5) (layer "B.Cu") (net 34))
+  (via (at 98.9805 96.52) (size 1.4) (drill 0.4) (layers "F.Cu" "B.Cu") (net 34))
+  (segment (start 96.49 91.425) (end 95.265 91.425) (width 0.5) (layer "B.Cu") (net 34))
+  (segment (start 97.79 92.725) (end 96.49 91.425) (width 0.5) (layer "B.Cu") (net 34))
   (segment (start 114.8175 96.52) (end 109.22 96.52) (width 0.5) (layer "B.Cu") (net 34))
-  (segment (start 97.79 91.44) (end 97.79 96.52) (width 0.5) (layer "B.Cu") (net 34))
+  (segment (start 98.9805 96.52) (end 97.79 95.3295) (width 0.5) (layer "B.Cu") (net 34))
+  (segment (start 97.79 95.3295) (end 97.79 92.725) (width 0.5) (layer "B.Cu") (net 34))
   (segment (start 113.020123 99.069877) (end 114.309877 99.069877) (width 0.5) (layer "B.Cu") (net 35))
   (segment (start 108.005667 104.084333) (end 113.020123 99.069877) (width 0.5) (layer "B.Cu") (net 35))

Commit message: Minor fixes
Parts:
- moved C4 14.5 mm to (151.2, 85.1), turned to 0 degrees
- moved C3 5.08 mm to (154.9, 91.4), turned to -90 degrees
- moved J3 2.54 mm to (152.4, 114.3)
- moved H1 2.54 mm to (154.9, 73.7)
- moved H4 2.54 mm to (154.9, 129.5)
- moved J4 1.80 mm to (99.1, 128.3)
Connections:
- U1 pad 2: unconnected-(U1-Pad2) -> B1-Y
- U1 pad 3: B1-Y -> B0-Y
- U1 pad 4: B0-Y -> A2-Y
- U1 pad 5: A2-Y -> A1-Y
- U1 pad 6: A1-Y -> A0-Y
- U1 pad 7: A0-Y -> B1-X
- U2 pad 15: B1-X -> unconnected-(U2-Pad15)
Routing:
- net Vin: track 228.1 -> 212.0 mm
- net B1-X: track 23.2 -> 15.1 mm, vias 2 -> 0
- net Net-(U1-Pad9): track 22.3 -> 15.5 mm
- net Net-(J1-Pad29): track 35.4 -> 29.6 mm
- net CFG-2: track 7.75 -> 5.21 mm
- net CFG-1: track 7.75 -> 5.21 mm
- net CFG-0: track 7.75 -> 5.21 mm
- net B1-Y: track 12.4 -> 14.6 mm
- net A2-Y: track 12.4 -> 14.6 mm
- net A1-Y: track 12.4 -> 14.6 mm
- net A0-Y: track 12.4 -> 14.6 mm
- net B0-Y: track 12.4 -> 14.6 mm
- net Net-(A1-Pad15): track 87.0 -> 85.1 mm
- net DATA-X: track 44.8 -> 43.1 mm
- net GND: track 52.1 -> 51.0 mm, vias 10 -> 8
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Other:
- board size 78.7 x 66 mm -> 76.2 x 66 mm
