File: Driver-boards/FlipDot34Nano/schematic/FlipDot34Nano/FlipDot34Nano.kicad_sch (KiCad schematic)
At the start: 15 parts, among them J1 FlipDot matrix, J2 I2C bus, J3 Config Jumpers, J4 Power 24V, U1 74HC595, U2 74HC595

Commit message: Refactoring
Parts:
- removed H3: MountingHole, MountingHole:MountingHole_3.2mm_M3, symbol Mechanical:MountingHole
- removed J3: Config Jumpers, Connector_PinHeader_2.54mm:PinHeader_2x03_P2.54mm_Vertical, symbol Connector_Generic:Conn_02x03_Odd_Even
- added C5: 100n, Capacitor_THT:C_Disc_D5.0mm_W2.5mm_P5.00mm, symbol Device:C_Small
- added D1: 1N5819, Diode_THT:D_DO-41_SOD81_P10.16mm_Horizontal, symbol Diode:1N5819
- added SW1: SW_DIP_x03, Button_Switch_THT:SW_DIP_SPSTx03_Slide_9.78x9.8mm_W7.62mm_P2.54mm, symbol Switch:SW_DIP_x03
- added U3: 74HC595, Package_DIP:DIP-16_W7.62mm_LongPads, symbol 74xx:74HC595
- C3: footprint Capacitor_THT:CP_Radial_D6.3mm_P2.50mm -> Capacitor_THT:CP_Radial_D8.0mm_P3.50mm
- renumbered H4 to H3, J4 to J3
Connections:
- net +5V: now also U1.10 (~{SRCLR}), U2.10 (~{SRCLR}), C5.2, U3.10 (~{SRCLR}), U3.16 (VCC); no longer U1.13 (~{OE}), U2.13 (~{OE})
- net A0-X: now also U3.4 (QE); no longer U2.4 (QE)
- net A0-Y: now also U2.6 (QG); no longer U1.6 (QG)
- net A1-X: now also U3.3 (QD); no longer U2.3 (QD)
- net A1-Y: now also U2.5 (QF); no longer U1.5 (QF)
- net A2-X: now also U3.2 (QC); no longer U2.2 (QC)
- net A2-Y: now also U2.4 (QE); no longer U1.4 (QE)
- net B0-X: now also U3.1 (QB); no longer U2.1 (QB)
- net B0-Y: now also U2.3 (QD); no longer U1.3 (QD)
- net B1-X: now also U2.7 (QH); no longer U1.7 (QH)
- net B1-Y: now also U2.2 (QC); no longer U1.2 (QC)
- net CFG-0: now also SW1.3
- net CFG-1: now also SW1.2
- net CFG-2: now also SW1.1
- net DATA-X: now also U3.5 (QF); no longer U2.5 (QF)
- net ENABLE-X-1: now also U1.15 (QA); no longer A1.5 (D2)
- net ENABLE-X-2: now also U1.1 (QB); no longer A1.6 (D3)
- net ENABLE-X-3: now also U1.2 (QC); no longer A1.7 (D4)
- net ENABLE-X-4: now also U1.3 (QD); no longer A1.8 (D5)
- net ENABLE-X-5: now also U1.4 (QE); no longer A1.9 (D6)
- net ENABLE-X-6: now also U1.5 (QF); no longer A1.10 (D7)
- net ENABLE-X-7: now also U1.6 (QG); no longer A1.11 (D8)
- net ENABLE-X-8: now also U1.7 (QH); no longer A1.12 (D9)
- net ENABLE-Y-RESET: now also U3.7 (QH); no longer U2.7 (QH)
- net ENABLE-Y-SET: now also U3.6 (QG); no longer U2.6 (QG)
- net GND: now also U1.13 (~{OE}), U2.13 (~{OE}), C5.1, D1.2 (A), SW1.4, SW1.5, SW1.6, U3.13 (~{OE}), U3.8 (GND); no longer J3.2 (Pin_2), U1.10 (~{SRCLR}), U2.10 (~{SRCLR})
- net at U1.11 (SRCLK), U2.11 (SRCLK): now also A1.9 (D6), U3.11 (SRCLK); no longer A1.14 (D11)
- net at U1.12 (RCLK), U2.12 (RCLK): now also A1.8 (D5), U3.12 (RCLK); no longer A1.15 (D12)
- net at U1.14 (SER): now also A1.6 (D3); no longer A1.13 (D10)
- net at U2.9 (QH'): now also U3.14 (SER)
- new net: D1.1 (K), J3.2 (Pin_2)
- no-connect marks 15 -> 23
Other:
- title: FlipDot34 Controller -> FlipDot34-Nano Controller Board
- moved on the sheet: C3, C4, H1, H2, H3, J2, J3
