File: schematic/34pin-matrix/34pin-matrix.kicad_sch (KiCad schematic)
At the start: 2 parts, among them J1 Input, J2 Input

Commit message: Refactoring
Parts:
- J2: value Input -> Output
Connections:
- net ENABLE-Y1 renamed ENABLE-Y-RESET
- net ENABLE-Y2 renamed ENABLE-Y-SET
- net M1 renamed ENABLE-X-1
- net M2 renamed ENABLE-X-2
- net M3 renamed ENABLE-X-3
- net M4 renamed ENABLE-X-4
- net M5 renamed ENABLE-X-5
- net M6 renamed ENABLE-X-6
- net M7 renamed ENABLE-X-7
- net M8 renamed ENABLE-X-8
Changed lines of the file:
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@@
     (stroke (width 0) (type default) (color 0 0 0 0))
   )
-  (wire (pts (xy 85.09 53.34) (xy 85.09 69.85))
+  (wire (pts (xy 87.63 53.34) (xy 87.63 69.85))
     (stroke (width 0) (type default) (color 0 0 0 0))
   )
@@
     (stroke (width 0) (type default) (color 0 0 0 0))
   )
-  (wire (pts (xy 64.77 53.34) (xy 85.09 53.34))
+  (wire (pts (xy 64.77 53.34) (xy 87.63 53.34))
     (stroke (width 0) (type default) (color 0 0 0 0))
   )
@@
     (stroke (width 0) (type default) (color 0 0 0 0))
   )
-  (wire (pts (xy 85.09 69.85) (xy 118.11 69.85))
+  (wire (pts (xy 87.63 69.85) (xy 118.11 69.85))
     (stroke (width 0) (type default) (color 0 0 0 0))
   )
@@
     (effects (font (size 1.27 1.27)) (justify right bottom))
   )
-  (label "M3" (at 121.92 55.88 0)
+  (label "ENABLE-X-3" (at 121.92 55.88 0)
     (effects (font (size 1.27 1.27)) (justify left bottom))
   )
@@
     (effects (font (size 1.27 1.27)) (justify left bottom))
   )
-  (label "M5" (at 71.12 63.5 0)
-    (effects (font (size 1.27 1.27)) (justify left bottom))
-  )
-  (label "M8" (at 121.92 68.58 0)
+  (label "ENABLE-X-5" (at 71.12 63.5 0)
+    (effects (font (size 1.27 1.27)) (justify left bottom))
+  )
+  (label "ENABLE-X-8" (at 121.92 68.58 0)
     (effects (font (size 1.27 1.27)) (justify left bottom))
   )
@@
     (effects (font (size 1.27 1.27)) (justify right bottom))
   )
-  (label "M8" (at 71.12 71.12 0)
+  (label "ENABLE-X-8" (at 71.12 71.12 0)
     (effects (font (size 1.27 1.27)) (justify left bottom))
   )
@@
     (effects (font (size 1.27 1.27)) (justify left bottom))
   )
-  (label "M2" (at 71.12 55.88 0)
-    (effects (font (size 1.27 1.27)) (justify left bottom))
-  )
-  (label "M3" (at 71.12 58.42 0)
+  (label "ENABLE-X-2" (at 71.12 55.88 0)
+    (effects (font (size 1.27 1.27)) (justify left bottom))
+  )
+  (label "ENABLE-X-3" (at 71.12 58.42 0)
     (effects (font (size 1.27 1.27)) (justify left bottom))
   )
@@
     (effects (font (size 1.27 1.27)) (justify left bottom))
   )
-  (label "ENABLE-Y1" (at 71.12 50.8 0)
+  (label "ENABLE-Y-RESET" (at 71.12 50.8 0)
     (effects (font (size 1.27 1.27)) (justify left bottom))
   )
@@
     (effects (font (size 1.27 1.27)) (justify right bottom))
   )
-  (label "M6" (at 71.12 66.04 0)
+  (label "ENABLE-X-6" (at 71.12 66.04 0)
     (effects (font (size 1.27 1.27)) (justify left bottom))
   )
@@
     (effects (font (size 1.27 1.27)) (justify right bottom))
   )
-  (label "M7" (at 71.12 68.58 0)
+  (label "ENABLE-X-7" (at 71.12 68.58 0)
     (effects (font (size 1.27 1.27)) (justify left bottom))
   )
@@
     (effects (font (size 1.27 1.27)) (justify left bottom))
   )
-  (label "M6" (at 121.92 63.5 0)
+  (label "ENABLE-X-6" (at 121.92 63.5 0)
     (effects (font (size 1.27 1.27)) (justify left bottom))
   )
@@
     (effects (font (size 1.27 1.27)) (justify right bottom))
   )
-  (label "M1" (at 121.92 71.12 0)
+  (label "ENABLE-X-1" (at 121.92 71.12 0)
     (effects (font (size 1.27 1.27)) (justify left bottom))
   )
@@
     (effects (font (size 1.27 1.27)) (justify right bottom))
   )
-  (label "M7" (at 121.92 66.04 0)
+  (label "ENABLE-X-7" (at 121.92 66.04 0)
     (effects (font (size 1.27 1.27)) (justify left bottom))
   )
@@
     (effects (font (size 1.27 1.27)) (justify right bottom))
   )
-  (label "ENABLE-Y1" (at 121.92 50.8 0)
-    (effects (font (size 1.27 1.27)) (justify left bottom))
-  )
-  (label "M1=ENABLE-X" (at 71.12 53.34 0)
+  (label "ENABLE-Y-RESET" (at 121.92 50.8 0)
+    (effects (font (size 1.27 1.27)) (justify left bottom))
+  )
+  (label "ENABLE-X-1" (at 71.12 53.34 0)
     (effects (font (size 1.27 1.27)) (justify left bottom))
   )
@@
     (effects (font (size 1.27 1.27)) (justify right bottom))
   )
-  (label "M4" (at 71.12 60.96 0)
-    (effects (font (size 1.27 1.27)) (justify left bottom))
-  )
-  (label "M5" (at 121.92 60.96 0)
+  (label "ENABLE-X-4" (at 71.12 60.96 0)
+    (effects (font (size 1.27 1.27)) (justify left bottom))
+  )
+  (label "ENABLE-X-5" (at 121.92 60.96 0)
     (effects (font (size 1.27 1.27)) (justify left bottom))
   )
@@
     (effects (font (size 1.27 1.27)) (justify right bottom))
   )
-  (label "ENABLE-Y2" (at 121.92 48.26 0)
-    (effects (font (size 1.27 1.27)) (justify left bottom))
-  )
-  (label "M2" (at 121.92 53.34 0)
+  (label "ENABLE-Y-SET" (at 121.92 48.26 0)
+    (effects (font (size 1.27 1.27)) (justify left bottom))
+  )
+  (label "ENABLE-X-2" (at 121.92 53.34 0)
     (effects (font (size 1.27 1.27)) (justify left bottom))
   )
@@
     (effects (font (size 1.27 1.27)) (justify right bottom))
   )
-  (label "M4" (at 121.92 58.42 0)
-    (effects (font (size 1.27 1.27)) (justify left bottom))
-  )
-  (label "ENABLE-Y2" (at 71.12 48.26 0)
+  (label "ENABLE-X-4" (at 121.92 58.42 0)
+    (effects (font (size 1.27 1.27)) (justify left bottom))
+  )
+  (label "ENABLE-Y-SET" (at 71.12 48.26 0)
     (effects (font (size 1.27 1.27)) (justify left bottom))
   )
@@
     (in_bom yes) (on_board yes) (fields_autoplaced)
     (property "Reference" "J2" (id 0) (at 109.22 31.75 0))
-    (property "Value" "Input" (id 1) (at 109.22 34.29 0))
+    (property "Value" "Output" (id 1) (at 109.22 34.29 0))
     (property "Footprint" "" (id 2) (at 107.95 58.42 0)
       (effects (font (size 1.27 1.27)) hide)
@@
     )
     (path "/1651a986-40d8-4e8b-bfa9-021c1abe7cf0"
-      (reference "J2") (unit 1) (value "Input") (footprint "")
+      (reference "J2") (unit 1) (value "Output") (footprint "")
     )
   )
