File: MatrixControllers/FlipDot34Nano/schematic/FlipDot34NanoSMD/FlipDot34NanoSMD.kicad_sch (KiCad schematic)
At the start: 14 parts, among them J1 FlipDot matrix, J2 I2C bus, J3 Power 24V, SW1 SW_DIP_x03, U1 74HC595D, U2 74HC595D, U3 74HC595D

Commit message: Create MatrixControllerI2C example
Parts:
- C4: footprint Capacitor_THT:C_Disc_D5.0mm_W2.5mm_P5.00mm -> Capacitor_SMD:C_1206_3216Metric_Pad1.33x1.80mm_HandSolder
Changed lines of the file:
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@@
       (effects (font (size 1.27 1.27)) (justify left))
     )
-    (property "Footprint" "Capacitor_THT:C_Disc_D5.0mm_W2.5mm_P5.00mm" (id 2) (at 161.29 128.27 0)
+    (property "Footprint" "Capacitor_SMD:C_1206_3216Metric_Pad1.33x1.80mm_HandSolder" (id 2) (at 161.29 128.27 0)
       (effects (font (size 1.27 1.27)) hide)
     )
@@
     )
     (path "/6147f979-29f6-4d1a-acc7-1b1c29a6f8c8"
-      (reference "C4") (unit 1) (value "100n") (footprint "Capacitor_THT:C_Disc_D5.0mm_W2.5mm_P5.00mm")
+      (reference "C4") (unit 1) (value "100n") (footprint "Capacitor_SMD:C_1206_3216Metric_Pad1.33x1.80mm_HandSolder")
     )
     (path "/257839d7-7f0e-4240-9d05-81d11e0f2236"
