File: MatrixControllers/FlipDot34Nano/schematic/FlipDot34NanoSMD3/FlipDot34NanoSMD3.kicad_pcb (KiCad board)
At the start: 2 copper layers, 64.8 x 45.7 mm, 15 parts, among them J1 FlipDot matrix, J2 I2C bus, J3 Power 24V, SW1 SW_DIP_x03, U1 74HC595D, U2 74HC595D, U3 74HC595D

Commit message: Bad Apple demo
Parts:
- added J4: RST, Connector_PinHeader_2.54mm:PinHeader_1x02_P2.54mm_Vertical, F.Cu at (85.1, 82.5)
- moved C4 3.24 mm to (96.5, 90.2)
- moved D2 1.27 mm to (85.1, 77.5)
- moved C1 0.90 mm to (71.9, 67.3)
- moved A1 0.64 mm to (76.2, 68.6)
Connections:
- J1 pad 5: Vin -> +5V
- J1 pad 6: Vin -> +5V
- J2 pad 1: RESET -> Net-(J2-Pad1)
Routing:
- net Vin: track 98.8 -> 49.1 mm
- net Net-(J2-Pad1): track 0.00 -> 27.5 mm
- net RESET: track 39.7 -> 12.3 mm
- net +5V: track 101.6 -> 122.0 mm
- net Net-(A1-Pad6): track 17.3 -> 19.8 mm
- net GND: track 24.8 -> 24.1 mm
- net SDA: track 20.7 -> 21.3 mm
