File: MatrixControllers/FlipDot34Nano/schematic/FlipDot34NanoSMD3/FlipDot34NanoSMD3.kicad_sch (KiCad schematic)
At the start: 14 parts, among them J1 FlipDot matrix, J2 I2C bus, J3 Power 24V, SW1 SW_DIP_x03, U1 74HC595D, U2 74HC595D, U3 74HC595D

Commit message: Bad Apple demo
Parts:
- added D2: 1N5817, Diode_THT:D_DO-41_SOD81_P10.16mm_Horizontal, symbol Diode:1N5819
- added J4: RST, Connector_PinHeader_2.54mm:PinHeader_1x02_P2.54mm_Vertical, symbol Connector:Conn_01x02_Male
Connections:
- net +5V: now also D2.1 (K); no longer C4.1, C5.1, J2.7 (Pin_7), J2.9 (Pin_9)
- net RESET: now also J4.2 (Pin_2); no longer J2.1 (Pin_1)
- new net: J2.1 (Pin_1), J4.1 (Pin_1)
- new net Vin: C4.1, C5.1, D2.2 (A), J2.7 (Pin_7), J2.9 (Pin_9)
Changed lines of the file:
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@@
   (junction (at 100.33 109.22) (diameter 0) (color 0 0 0 0)
   )
-  (junction (at 49.53 101.6) (diameter 0) (color 0 0 0 0)
-  )
   (junction (at 158.75 36.83) (diameter 0) (color 0 0 0 0)
   )
@@
   )
   (junction (at 87.63 120.65) (diameter 0) (color 0 0 0 0)
+  )
+  (junction (at 49.53 102.87) (diameter 0) (color 0 0 0 0)
   )
   (junction (at 87.63 118.11) (diameter 0) (color 0 0 0 0)
@@
     (stroke (width 0) (type default) (color 0 0 0 0))
   )
+  (wire (pts (xy 46.99 102.87) (xy 49.53 102.87))
+    (stroke (width 0) (type default) (color 0 0 0 0))
+  )
   (wire (pts (xy 158.75 36.83) (xy 158.75 39.37))
     (stroke (width 0) (type default) (color 0 0 0 0))
@@
     (stroke (width 0) (type default) (color 0 0 0 0))
   )
-  (wire (pts (xy 49.53 101.6) (xy 49.53 102.87))
+  (wire (pts (xy 49.53 100.33) (xy 49.53 102.87))
     (stroke (width 0) (type default) (color 0 0 0 0))
   )
@@
     (stroke (width 0) (type default) (color 0 0 0 0))
   )
+  (wire (pts (xy 149.86 40.64) (xy 149.86 41.91))
+    (stroke (width 0) (type default) (color 0 0 0 0))
+  )
   (wire (pts (xy 100.33 57.15) (xy 100.33 71.12))
     (stroke (width 0) (type default) (color 0 0 0 0))
@@
     (stroke (width 0) (type default) (color 0 0 0 0))
   )
+  (wire (pts (xy 166.37 115.57) (xy 170.18 115.57))
+    (stroke (width 0) (type default) (color 0 0 0 0))
+  )
   (wire (pts (xy 153.67 67.31) (xy 158.75 67.31))
     (stroke (width 0) (type default) (color 0 0 0 0))
@@
     (stroke (width 0) (type default) (color 0 0 0 0))
   )
-  (wire (pts (xy 167.64 115.57) (xy 170.18 115.57))
-    (stroke (width 0) (type default) (color 0 0 0 0))
-  )
   (wire (pts (xy 87.63 41.91) (xy 102.87 41.91))
     (stroke (width 0) (type default) (color 0 0 0 0))
@@
     (stroke (width 0) (type default) (color 0 0 0 0))
   )
+  (wire (pts (xy 157.48 115.57) (xy 163.83 115.57))
+    (stroke (width 0) (type default) (color 0 0 0 0))
+  )
   (wire (pts (xy 93.98 46.99) (xy 93.98 74.93))
     (stroke (width 0) (type default) (color 0 0 0 0))
@@
     (stroke (width 0) (type default) (color 0 0 0 0))
   )
+  (wire (pts (xy 35.56 102.87) (xy 39.37 102.87))
+    (stroke (width 0) (type default) (color 0 0 0 0))
+  )
   (wire (pts (xy 123.19 52.07) (xy 125.73 52.07))
     (stroke (width 0) (type default) (color 0 0 0 0))
@@
     (stroke (width 0) (type default) (color 0 0 0 0))
   )
-  (wire (pts (xy 35.56 101.6) (xy 49.53 101.6))
-    (stroke (width 0) (type default) (color 0 0 0 0))
-  )
   (wire (pts (xy 171.45 36.83) (xy 187.96 36.83))
     (stroke (width 0) (type default) (color 0 0 0 0))
@@
     (stroke (width 0) (type default) (color 0 0 0 0))
   )
-  (wire (pts (xy 49.53 100.33) (xy 49.53 101.6))
-    (stroke (width 0) (type default) (color 0 0 0 0))
-  )
   (wire (pts (xy 93.98 74.93) (xy 93.98 99.06))
     (stroke (width 0) (type default) (color 0 0 0 0))
@@
     )
   )
-  (global_label "RESET" (shape input) (at 167.64 115.57 180) (fields_autoplaced)
-    (effects (font (size 1 1)) (justify right))
-    (property "Intersheet References" "${INTERSHEET_REFS}" (id 0) (at 161.2162 115.5075 0)
+  (global_label "RESET" (shape input) (at 157.48 115.57 180) (fields_autoplaced)
+    (effects (font (size 1 1)) (justify right))
+    (property "Intersheet References" "${INTERSHEET_REFS}" (id 0) (at 151.0562 115.5075 0)
       (effects (font (size 1 1)) (justify right) hide)
     )
@@
     )
   )
-  (global_label "Vin" (shape input) (at 35.56 101.6 180) (fields_autoplaced)
-    (effects (font (size 1 1)) (justify right))
-    (property "Intersheet References" "${INTERSHEET_REFS}" (id 0) (at 31.4219 101.5375 0)
+  (global_label "Vin" (shape input) (at 35.56 102.87 180) (fields_autoplaced)
+    (effects (font (size 1 1)) (justify right))
+    (property "Intersheet References" "${INTERSHEET_REFS}" (id 0) (at 31.4219 102.8075 0)
       (effects (font (size 1 1)) (justify right) hide)
     )
@@
     (pin "9")
   )
-  (symbol (lib_id "power:+5V") (at 149.86 41.91 0) (unit 1)
-    (in_bom yes) (on_board yes) (fields_autoplaced)
-    (property "Reference" "#PWR013" (id 0) (at 149.86 45.72 0)
-      (effects (font (size 1.27 1.27)) hide)
-    )
-    (property "Value" "+5V" (id 1) (at 149.86 36.83 0))
-    (property "Footprint" "" (id 2) (at 149.86 41.91 0)
-      (effects (font (size 1.27 1.27)) hide)
-    )
-    (property "Datasheet" "" (id 3) (at 149.86 41.91 0)
-      (effects (font (size 1.27 1.27)) hide)
-    )
-    (pin "1")
-  )
   (symbol (lib_id "power:GND") (at 113.03 123.19 0) (unit 1)
     (in_bom yes) (on_board yes) (fields_autoplaced)
@@
     )
     (property "Datasheet" "~" (id 3) (at 156.21 128.27 0)
+      (effects (font (size 1.27 1.27)) hide)
+    )
+    (pin "1")
+    (pin "2")
+  )
+  (symbol (lib_id "Diode:1N5819") (at 43.18 102.87 180) (unit 1)
+    (in_bom yes) (on_board yes) (fields_autoplaced)
+    (property "Reference" "D2" (id 0) (at 43.4975 96.52 0))
+    (property "Value" "1N5817" (id 1) (at 43.4975 99.06 0))
+    (property "Footprint" "Diode_THT:D_DO-41_SOD81_P10.16mm_Horizontal" (id 2) (at 43.18 98.425 0)
+      (effects (font (size 1.27 1.27)) hide)
+    )
+    (property "Datasheet" "http://www.vishay.com/docs/88525/1n5817.pdf" (id 3) (at 43.18 102.87 0)
       (effects (font (size 1.27 1.27)) hide)
     )
@@
     (pin "9")
   )
+  (symbol (lib_id "power:+5V") (at 149.86 40.64 0) (unit 1)
+    (in_bom yes) (on_board yes) (fields_autoplaced)
+    (property "Reference" "#PWR?" (id 0) (at 149.86 44.45 0)
+      (effects (font (size 1.27 1.27)) hide)
+    )
+    (property "Value" "+5V" (id 1) (at 149.86 35.56 0))
+    (property "Footprint" "" (id 2) (at 149.86 40.64 0)
+      (effects (font (size 1.27 1.27)) hide)
+    )
+    (property "Datasheet" "" (id 3) (at 149.86 40.64 0)
+      (effects (font (size 1.27 1.27)) hide)
+    )
+    (pin "1")
+  )
+  (symbol (lib_id "Connector:Conn_01x02_Male") (at 166.37 110.49 270) (unit 1)
+    (in_bom yes) (on_board yes)
+    (property "Reference" "J4" (id 0) (at 160.02 109.22 90)
+      (effects (font (size 1.27 1.27)) (justify right))
+    )
+    (property "Value" "RST" (id 1) (at 161.29 111.76 90)
+      (effects (font (size 1.27 1.27)) (justify right))
+    )
+    (property "Footprint" "Connector_PinHeader_2.54mm:PinHeader_1x02_P2.54mm_Vertical" (id 2) (at 166.37 110.49 0)
+      (effects (font (size 1.27 1.27)) hide)
+    )
+    (property "Datasheet" "~" (id 3) (at 166.37 110.49 0)
+      (effects (font (size 1.27 1.27)) hide)
+    )
+    (pin "1")
+    (pin "2")
+  )
   (symbol (lib_id "Device:C_Small") (at 101.6 31.75 90) (unit 1)
     (in_bom yes) (on_board yes)
@@
       (reference "#PWR012") (unit 1) (value "GND") (footprint "")
     )
-    (path "/0c18d6c5-f1fc-4a30-83ba-9522edfac149"
-      (reference "#PWR013") (unit 1) (value "+5V") (footprint "")
-    )
     (path "/2e5e3102-fdb9-450c-b6fe-ef609f13cefe"
       (reference "#PWR014") (unit 1) (value "GND") (footprint "")
@@
       (reference "#PWR0105") (unit 1) (value "+5V") (footprint "")
     )
+    (path "/8bd21d15-4278-4bfb-9081-da5dec67eaa5"
+      (reference "#PWR?") (unit 1) (value "+5V") (footprint "")
+    )
     (path "/52f68f8d-08cf-41ba-aaf3-dd276fb02dbd"
       (reference "A1") (unit 1) (value "Arduino_Nano_v3.x") (footprint "Module:Arduino_Nano")
@@
       (reference "D1") (unit 1) (value "1N5819") (footprint "Diode_THT:D_DO-41_SOD81_P10.16mm_Horizontal")
     )
+    (path "/2d24f90a-d5c6-465c-8871-4c80385fcc66"
+      (reference "D2") (unit 1) (value "1N5817") (footprint "Diode_THT:D_DO-41_SOD81_P10.16mm_Horizontal")
+    )
     (path "/51498787-d262-4042-a222-87c9237f3cab"
       (reference "J1") (unit 1) (value "FlipDot matrix") (footprint "Connector_PinSocket_2.54mm:PinSocket_2x17_P2.54mm_Vertical")
@@
       (reference "J3") (unit 1) (value "Power 24V") (footprint "TerminalBlock:TerminalBlock_bornier-2_P5.08mm")
     )
+    (path "/926cc1ad-5eb7-4bb0-b857-514ecb6a4b69"
+      (reference "J4") (unit 1) (value "RST") (footprint "Connector_PinHeader_2.54mm:PinHeader_1x02_P2.54mm_Vertical")
+    )
     (path "/d66451d9-0ea8-410b-8ebe-f019fe924330"
