File: MatrixControllers/FlipDot34Nano/schematic/FlipDot34-Nano-TwoSides-V3/FlipDot34-Nano-TwoSides-V3.kicad_sch (KiCad schematic)
At the start: 14 parts, among them J1 FlipDot matrix, J2 I2C bus, J3 Power 24V, SW1 SW_DIP_x03, U1 74HC595D, U2 74HC595D, U3 74HC595D

Commit message: Refactoring
Parts:
- added C6: 100n, Capacitor_SMD:C_1206_3216Metric_Pad1.33x1.80mm_HandSolder, symbol Device:C_Small
- added D2, D4: RB160M, Diode_SMD:D_SOD-123, symbol Diode:1N5819
- added D3: 1N5819, Diode_THT:D_DO-41_SOD81_P10.16mm_Horizontal, symbol Diode:1N5819
- added J4: RST, Connector_PinHeader_2.54mm:PinHeader_1x02_P2.54mm_Vertical, symbol Connector:Conn_01x02_Male
- added J5: Barrel_Jack, Connector_BarrelJack:BarrelJack_Wuerth_6941xx301002, symbol Connector:Barrel_Jack
- added J6: Shift, Connector_PinHeader_2.54mm:PinHeader_1x05_P2.54mm_Vertical, symbol Connector:Conn_01x05_Pin
- added J7: I2C, Connector_PinHeader_2.54mm:PinHeader_1x04_P2.54mm_Vertical, symbol Connector:Conn_01x04_Pin
- added J8: DC-DC, Connector_PinHeader_2.54mm:PinHeader_1x04_P2.54mm_Vertical, symbol Connector:Conn_01x04_Pin
- added R1: 100k, Resistor_SMD:R_1206_3216Metric, symbol Device:R
Connections:
- net +5V: now also D2.1 (K), D4.1 (K), J6.4 (Pin_4), J7.3 (Pin_3), R1.1; no longer C4.1, J2.7 (Pin_7), J2.9 (Pin_9)
- net CFG-0: now also SW1.1; no longer SW1.3
- net CFG-2: now also SW1.3; no longer SW1.1
- net GND: now also J3.2 (Pin_2), C6.1, J5.2, J6.5 (Pin_5), J7.4 (Pin_4), J8.2 (Pin_2); no longer D1.2 (A)
- net RESET: now also J4.2 (Pin_2), R1.2; no longer J2.1 (Pin_1)
- net SCL: now also J7.2 (Pin_2)
- net SDA: now also J7.1 (Pin_1)
- net at A1.9 (D6), U1.11 (SRCLK), U2.11 (SRCLK)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: now also J6.1 (Pin_1)
- net at A1.8 (D5), U1.12 (RCLK), U2.12 (RCLK)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: now also J6.2 (Pin_2)
- net at A1.6 (D3), U1.14 (SER): now also J6.3 (Pin_3)
- net 24V+: now reaches J1.29 (Pin_29), J1.30 (Pin_30)
- net 24V+: now also D1.1 (K), D3.1 (K), J8.3 (Pin_3); no longer J3.1 (Pin_1)
- new net: D3.2 (A), J5.1
- new net: D1.2 (A), J3.1 (Pin_1)
- new net: J2.1 (Pin_1), J4.1 (Pin_1)
- new net V0+: C6.2, D4.2 (A), J8.1 (Pin_1)
- new net Vin: C4.1, D2.2 (A), J2.7 (Pin_7), J2.9 (Pin_9)
- no-connect marks 23 -> 24
Other:
- moved on the sheet: C4, C5, D1, J2, J3
